File: corne-classic/pcb/corne-classic.kicad_pcb (KiCad board)
At the start: 2 copper layers, 133.8 x 92.2 mm, 98 parts, among them J1 MJ-4PP-9, J2 OLED, J3 LED, P1 i2c-pin, P2 i2c-pin, SW1 SW_PUSH, SW10 SW_PUSH, SW11 SW_PUSH, SW12 SW_PUSH, SW13 SW_PUSH, SW14 SW_PUSH, SW15 SW_PUSH, SW16 SW_PUSH, SW17 SW_PUSH, SW18 SW_PUSH, SW19 SW_PUSH, SW2 SW_PUSH, SW20 SW_PUSH, SW21 SW_PUSH, SW3 SW_PUSH, SW4 SW_PUSH, SW5 SW_PUSH, SW6 SW_PUSH, SW7 SW_PUSH, SW8 SW_PUSH, SW9 SW_PUSH, U1 ProMicro

Commit message: first commit
Parts:
- removed ? (x9): , kbd:LEGO_HOLE
- removed G*** (x2): LOGO, kbd:corne
- removed JP1: , kbd:JPC2
- added D22: D, kbd:D3_TH_SMD, F.Cu at (42.9, 90.9)
- added L28: SK6812MINI, kbd:SK6812MINI_rev, F.Cu at (51.0, 85.6)
- added SW22: SW_PUSH, kbd:MX_ALPS_PG1350_noLed, F.Cu at (51.0, 91.0)
- RSW1: value Reset -> SW_PUSH
Connections:
- J1 pad B: Net-(J1-PadB) -> data
- P2 pad 1: Net-(J1-PadB) -> data
Routing:
- net row3: track 121.8 -> 249.7 mm, vias 3 -> 6
- net VCC: track 758.8 -> 802.4 mm
- net col0: track 245.7 -> 280.4 mm, vias 4 -> 5
- net Net-(L19-Pad1): track 5.40 -> 37.8 mm, vias 1 -> 2
- net GND: track 797.7 -> 826.8 mm, vias 49 -> 50
- net data: track 55.3 -> 75.1 mm, vias 4 -> 5
- net Net-(J1-PadB): track 18.9 -> 0.00 mm, vias 1 -> 0
- net Net-(D22-Pad2): track 0.00 -> 14.0 mm
- net col3: track 225.1 -> 229.7 mm
- net col5: track 187.0 -> 191.4 mm
- net col4: track 194.3 -> 198.4 mm
- net Net-(L28-Pad1): track 0.00 -> 4.02 mm, vias 0 -> 1
- net col2: track 197.5 -> 200.7 mm
- net col1: track 221.3 -> 224.5 mm
- net Net-(L23-Pad1): track 49.6 -> 50.7 mm
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- removed copper zone on B.Cu, net GND
- removed copper zone on F.Cu, net GND
Other:
- board size 133.8 x 92.2 mm -> 152.8 x 92.2 mm
- board text added: "Jorne Classic v2.0 PCB Designed by foostan & Joric"
- board text removed: "Corne Classic v2.0 PCB Designed by foostan"
