File: corne-cherry/pcb/corne-cherry.sch (KiCad schematic (older format))
At the start: 87 parts, among them J1 MJ-4PP-9, J2 OLED, J3 LED, P1 i2c-pin, P2 i2c-pin, SW1 SW_PUSH, SW10 SW_PUSH, SW11 SW_PUSH, SW12 SW_PUSH, SW13 SW_PUSH, SW14 SW_PUSH, SW15 SW_PUSH, SW16 SW_PUSH, SW17 SW_PUSH, SW18 SW_PUSH, SW19 SW_PUSH, SW2 SW_PUSH, SW20 SW_PUSH, SW21 SW_PUSH, SW3 SW_PUSH, SW4 SW_PUSH, SW5 SW_PUSH, SW6 SW_PUSH, SW7 SW_PUSH, SW8 SW_PUSH, SW9 SW_PUSH, U1 ProMicro

Commit message: added drawings
Parts:
- added D22: D, kbd:D3_SMD, symbol Device:D
- added G01, G02: Logo_Open_Hardware_Small, kbd:corne, symbol Graphic:Logo_Open_Hardware_Small
- added H1, H2, H3, H4, H5, H6, H7, H8, H9: MountingHole, kbd:LEGO_HOLE, symbol Mechanical:MountingHole
- added L28: SK6812MINI, kbd:SK6812MINI_rev, symbol corne-cherry-rescue:SK6812MINI-kbd
- added SW22: SW_PUSH, kbd:CherryMX_MidHeight_Hotswap, symbol corne-cherry-rescue:SW_PUSH-kbd
- J1: symbol kbd:MJ-4PP-9 -> corne-cherry-rescue:MJ-4PP-9-kbd
- L1, L10, L11, L12, L13, L14, L15, L16, L17, L18, L19, L2, L20, L21, L22, L23, L24, L25, L26, L27, L3, L4, L5, L6, L7, L8, L9: symbol kbd:SK6812MINI -> corne-cherry-rescue:SK6812MINI-kbd
- RSW1, SW1, SW10, SW11, SW12, SW13, SW14, SW15, SW16, SW17, SW18, SW19, SW2, SW20, SW3, SW4, SW5, SW6, SW7, SW8, SW9: symbol kbd:SW_PUSH -> corne-cherry-rescue:SW_PUSH-kbd
- SW21: footprint kbd:MX_ALPS_PG1350_noLed_1.75u -> kbd:CherryMX_MidHeight_Hotswap; symbol kbd:SW_PUSH -> corne-cherry-rescue:SW_PUSH-kbd
- U1: symbol kbd:ProMicro -> corne-cherry-rescue:ProMicro-kbd
Connections:
- wire segments 265 -> 274
