File: corne-cherry/pcb/corne-cherry.kicad_pcb (KiCad board)
At the start: 2 copper layers, 152.8 x 91.4 mm, 101 parts, among them J1 MJ-4PP-9, J2 OLED, J3 LED, P1 i2c-pin, P2 i2c-pin, SW1 SW_PUSH, SW10 SW_PUSH, SW11 SW_PUSH, SW12 SW_PUSH, SW13 SW_PUSH, SW14 SW_PUSH, SW15 SW_PUSH, SW16 SW_PUSH, SW17 SW_PUSH, SW18 SW_PUSH, SW19 SW_PUSH, SW2 SW_PUSH, SW20 SW_PUSH, SW21 SW_PUSH, SW22 SW_PUSH, SW3 SW_PUSH, SW4 SW_PUSH, SW5 SW_PUSH, SW6 SW_PUSH, SW7 SW_PUSH, SW8 SW_PUSH, SW9 SW_PUSH, U1 ProMicro

Commit message: updated corne-cherry
Routing:
- net row3: track 239.1 -> 246.2 mm
- net col2: track 205.6 -> 204.9 mm
Other:
- outline, holes or cut-outs redrawn
- net class Default: trace_width 0.25 -> 0.2
- net class Power added: clearance 0.2, trace_width 0.5, via_dia 0.6, via_drill 0.4
- rule pad_to_mask_clearance: 0.2 -> 0
