File: corne-cherry/pcb_wl/left/corne-cherry-left.sch (KiCad schematic (older format))
At the start: 50 parts, among them J1 MJ-4PP-9, J2 OLED, J3 Conn_01x02_Female, SW1 SW_PUSH, SW10 SW_PUSH, SW11 SW_PUSH, SW12 SW_PUSH, SW13 SW_PUSH, SW14 SW_PUSH, SW15 SW_PUSH, SW16 SW_PUSH, SW17 SW_PUSH, SW18 SW_PUSH, SW19 SW_PUSH, SW2 SW_PUSH, SW20 SW_PUSH, SW21 SW_PUSH, SW22 SW_PUSH, SW23 SW_SPDT, SW3 SW_PUSH, SW4 SW_PUSH, SW5 SW_PUSH, SW6 SW_PUSH, SW7 SW_PUSH, SW8 SW_PUSH, SW9 SW_PUSH, U1 ProMicro

Commit message: Small revision bump: bigger battery header, smaller footprints
Parts:
- J3: footprint Connector_PinHeader_2.00mm:PinHeader_1x02_P2.00mm_Vertical -> kbd:Battery_Header
- SW1, SW10, SW11, SW12, SW13, SW14, SW15, SW16, SW17, SW18, SW19, SW2, SW20, SW22, SW3, SW4, SW5, SW6, SW7, SW8, SW9: footprint kbd:CherryMX_Hotswap -> kbd:MX-Alps-HS-1U
- SW21: footprint kbd:CherryMX_Hotswap_1.5u -> kbd:MX-Alps-HS-1.5U
Changed lines of the file:
@@
 F 0 "SW2" H 4750 1385 50  0000 C CNN
 F 1 "SW_PUSH" H 4600 1195 50  0000 C CNN
-F 2 "kbd:CherryMX_Hotswap" H 4600 1275 50  0001 C CNN
+F 2 "kbd:MX-Alps-HS-1U" H 4600 1275 50  0001 C CNN
 F 3 "" H 4600 1275 50  0000 C CNN
 	1    4600 1275
@@
 F 0 "SW3" H 5450 1385 50  0000 C CNN
 F 1 "SW_PUSH" H 5300 1195 50  0000 C CNN
-F 2 "kbd:CherryMX_Hotswap" H 5300 1275 50  0001 C CNN
+F 2 "kbd:MX-Alps-HS-1U" H 5300 1275 50  0001 C CNN
 F 3 "" H 5300 1275 50  0000 C CNN
 	1    5300 1275
@@
 F 0 "SW4" H 6150 1385 50  0000 C CNN
 F 1 "SW_PUSH" H 6000 1195 50  0000 C CNN
-F 2 "kbd:CherryMX_Hotswap" H 6000 1275 50  0001 C CNN
+F 2 "kbd:MX-Alps-HS-1U" H 6000 1275 50  0001 C CNN
 F 3 "" H 6000 1275 50  0000 C CNN
 	1    6000 1275
@@
 F 0 "SW5" H 6850 1385 50  0000 C CNN
 F 1 "SW_PUSH" H 6700 1195 50  0000 C CNN
-F 2 "kbd:CherryMX_Hotswap" H 6700 1275 50  0001 C CNN
+F 2 "kbd:MX-Alps-HS-1U" H 6700 1275 50  0001 C CNN
 F 3 "" H 6700 1275 50  0000 C CNN
 	1    6700 1275
@@
 F 0 "SW6" H 7550 1385 50  0000 C CNN
 F 1 "SW_PUSH" H 7400 1195 50  0000 C CNN
-F 2 "kbd:CherryMX_Hotswap" H 7400 1275 50  0001 C CNN
+F 2 "kbd:MX-Alps-HS-1U" H 7400 1275 50  0001 C CNN
 F 3 "" H 7400 1275 50  0000 C CNN
 	1    7400 1275
@@
 F 0 "SW1" H 4050 1385 50  0000 C CNN
 F 1 "SW_PUSH" H 3900 1195 50  0000 C CNN
-F 2 "kbd:CherryMX_Hotswap" H 3900 1275 50  0001 C CNN
+F 2 "kbd:MX-Alps-HS-1U" H 3900 1275 50  0001 C CNN
 F 3 "" H 3900 1275 50  0000 C CNN
 	1    3900 1275
@@
 F 0 "SW8" H 4750 1985 50  0000 C CNN
 F 1 "SW_PUSH" H 4600 1795 50  0000 C CNN
-F 2 "kbd:CherryMX_Hotswap" H 4600 1875 50  0001 C CNN
+F 2 "kbd:MX-Alps-HS-1U" H 4600 1875 50  0001 C CNN
 F 3 "" H 4600 1875 50  0000 C CNN
 	1    4600 1875
@@
 F 0 "SW9" H 5450 1985 50  0000 C CNN
 F 1 "SW_PUSH" H 5300 1795 50  0000 C CNN
-F 2 "kbd:CherryMX_Hotswap" H 5300 1875 50  0001 C CNN
+F 2 "kbd:MX-Alps-HS-1U" H 5300 1875 50  0001 C CNN
 F 3 "" H 5300 1875 50  0000 C CNN
 	1    5300 1875
@@
 F 0 "SW10" H 6150 1985 50  0000 C CNN
 F 1 "SW_PUSH" H 6000 1795 50  0000 C CNN
-F 2 "kbd:CherryMX_Hotswap" H 6000 1875 50  0001 C CNN
+F 2 "kbd:MX-Alps-HS-1U" H 6000 1875 50  0001 C CNN
 F 3 "" H 6000 1875 50  0000 C CNN
 	1    6000 1875
@@
 F 0 "SW11" H 6850 1985 50  0000 C CNN
 F 1 "SW_PUSH" H 6700 1795 50  0000 C CNN
-F 2 "kbd:CherryMX_Hotswap" H 6700 1875 50  0001 C CNN
+F 2 "kbd:MX-Alps-HS-1U" H 6700 1875 50  0001 C CNN
 F 3 "" H 6700 1875 50  0000 C CNN
 	1    6700 1875
@@
 F 0 "SW12" H 7550 1985 50  0000 C CNN
 F 1 "SW_PUSH" H 7400 1795 50  0000 C CNN
-F 2 "kbd:CherryMX_Hotswap" H 7400 1875 50  0001 C CNN
+F 2 "kbd:MX-Alps-HS-1U" H 7400 1875 50  0001 C CNN
 F 3 "" H 7400 1875 50  0000 C CNN
 	1    7400 1875
@@
 F 0 "SW7" H 4050 1985 50  0000 C CNN
 F 1 "SW_PUSH" H 3900 1795 50  0000 C CNN
-F 2 "kbd:CherryMX_Hotswap" H 3900 1875 50  0001 C CNN
+F 2 "kbd:MX-Alps-HS-1U" H 3900 1875 50  0001 C CNN
 F 3 "" H 3900 1875 50  0000 C CNN
 	1    3900 1875
@@
 F 0 "SW14" H 4750 2585 50  0000 C CNN
 F 1 "SW_PUSH" H 4600 2395 50  0000 C CNN
-F 2 "kbd:CherryMX_Hotswap" H 4600 2475 50  0001 C CNN
+F 2 "kbd:MX-Alps-HS-1U" H 4600 2475 50  0001 C CNN
 F 3 "" H 4600 2475 50  0000 C CNN
 	1    4600 2475
@@
 F 0 "SW15" H 5450 2585 50  0000 C CNN
 F 1 "SW_PUSH" H 5300 2395 50  0000 C CNN
-F 2 "kbd:CherryMX_Hotswap" H 5300 2475 50  0001 C CNN
+F 2 "kbd:MX-Alps-HS-1U" H 5300 2475 50  0001 C CNN
 F 3 "" H 5300 2475 50  0000 C CNN
 	1    5300 2475
@@
 F 0 "SW16" H 6150 2585 50  0000 C CNN
 F 1 "SW_PUSH" H 6000 2395 50  0000 C CNN
-F 2 "kbd:CherryMX_Hotswap" H 6000 2475 50  0001 C CNN
+F 2 "kbd:MX-Alps-HS-1U" H 6000 2475 50  0001 C CNN
 F 3 "" H 6000 2475 50  0000 C CNN
 	1    6000 2475
@@
 F 0 "SW17" H 6850 2585 50  0000 C CNN
 F 1 "SW_PUSH" H 6700 2395 50  0000 C CNN
-F 2 "kbd:CherryMX_Hotswap" H 6700 2475 50  0001 C CNN
+F 2 "kbd:MX-Alps-HS-1U" H 6700 2475 50  0001 C CNN
 F 3 "" H 6700 2475 50  0000 C CNN
 	1    6700 2475
@@
 F 0 "SW18" H 7550 2585 50  0000 C CNN
 F 1 "SW_PUSH" H 7400 2395 50  0000 C CNN
-F 2 "kbd:CherryMX_Hotswap" H 7400 2475 50  0001 C CNN
+F 2 "kbd:MX-Alps-HS-1U" H 7400 2475 50  0001 C CNN
 F 3 "" H 7400 2475 50  0000 C CNN
 	1    7400 2475
@@
 F 0 "SW13" H 4050 2585 50  0000 C CNN
 F 1 "SW_PUSH" H 3900 2395 50  0000 C CNN
-F 2 "kbd:CherryMX_Hotswap" H 3900 2475 50  0001 C CNN
+F 2 "kbd:MX-Alps-HS-1U" H 3900 2475 50  0001 C CNN
 F 3 "" H 3900 2475 50  0000 C CNN
 	1    3900 2475
@@
 F 0 "SW20" H 6850 3185 50  0000 C CNN
 F 1 "SW_PUSH" H 6700 2995 50  0000 C CNN
-F 2 "kbd:CherryMX_Hotswap" H 6700 3075 50  0001 C CNN
+F 2 "kbd:MX-Alps-HS-1U" H 6700 3075 50  0001 C CNN
 F 3 "" H 6700 3075 50  0000 C CNN
 	1    6700 3075
@@
 F 0 "SW21" H 7550 3185 50  0000 C CNN
 F 1 "SW_PUSH" H 7400 2995 50  0000 C CNN
-F 2 "kbd:CherryMX_Hotswap_1.5u" H 7400 3075 50  0001 C CNN
+F 2 "kbd:MX-Alps-HS-1.5U" H 7400 3075 50  0001 C CNN
 F 3 "" H 7400 3075 50  0000 C CNN
 	1    7400 3075
@@
 F 0 "SW19" H 6150 3185 50  0000 C CNN
 F 1 "SW_PUSH" H 6000 2995 50  0000 C CNN
-F 2 "kbd:CherryMX_Hotswap" H 6000 3075 50  0001 C CNN
+F 2 "kbd:MX-Alps-HS-1U" H 6000 3075 50  0001 C CNN
 F 3 "" H 6000 3075 50  0000 C CNN
 	1    6000 3075
@@
 F 0 "J3" H 4938 3896 50  0000 L CNN
 F 1 "Conn_01x02_Female" H 4938 3805 50  0000 L CNN
-F 2 "Connector_PinHeader_2.00mm:PinHeader_1x02_P2.00mm_Vertical" H 4910 3920 50  0001 C CNN
+F 2 "kbd:Battery_Header" H 4910 3920 50  0001 C CNN
 F 3 "~" H 4910 3920 50  0001 C CNN
 	1    4910 3920
@@
 F 0 "SW22" H 4050 3185 50  0000 C CNN
 F 1 "SW_PUSH" H 3900 2995 50  0000 C CNN
-F 2 "kbd:CherryMX_Hotswap" H 3900 3075 50  0001 C CNN
+F 2 "kbd:MX-Alps-HS-1U" H 3900 3075 50  0001 C CNN
 F 3 "" H 3900 3075 50  0000 C CNN
 	1    3900 3075
