File: corne-cherry/pcb_wl/right/corne-cherry-right.sch (KiCad schematic (older format))
At the start: 50 parts, among them J3 MJ-4PP-9, J4 OLED, J5 Conn_01x02_Female, SW22 SW_PUSH, SW23 SW_PUSH, SW24 SW_PUSH, SW25 SW_PUSH, SW26 SW_PUSH, SW27 SW_PUSH, SW28 SW_PUSH, SW29 SW_PUSH, SW30 SW_PUSH, SW31 SW_PUSH, SW32 SW_PUSH, SW33 SW_PUSH, SW34 SW_PUSH, SW35 SW_PUSH, SW36 SW_PUSH, SW37 SW_PUSH, SW38 SW_PUSH, SW39 SW_PUSH, SW40 SW_PUSH, SW41 SW_PUSH, SW42 SW_PUSH, SW43 SW_PUSH, SW44 SW_SPDT, U2 ProMicro

Commit message: Small revision bump: bigger battery header, smaller footprints
Parts:
- J5: footprint Connector_PinHeader_2.00mm:PinHeader_1x02_P2.00mm_Vertical -> kbd:Battery_Header
- SW22, SW23, SW24, SW25, SW26, SW27, SW28, SW29, SW30, SW31, SW32, SW33, SW34, SW35, SW36, SW37, SW38, SW39, SW40, SW41, SW43: footprint kbd:CherryMX_Hotswap -> kbd:MX-Alps-HS-1U
- SW42: footprint kbd:CherryMX_Hotswap_1.5u -> kbd:MX-Alps-HS-1.5U
Changed lines of the file:
@@
 F 0 "SW23" H 12725 1510 50  0000 C CNN
 F 1 "SW_PUSH" H 12575 1320 50  0000 C CNN
-F 2 "kbd:CherryMX_Hotswap" H 12575 1400 50  0001 C CNN
+F 2 "kbd:MX-Alps-HS-1U" H 12575 1400 50  0001 C CNN
 F 3 "" H 12575 1400 50  0000 C CNN
 	1    12575 1400
@@
 F 0 "SW24" H 13425 1510 50  0000 C CNN
 F 1 "SW_PUSH" H 13275 1320 50  0000 C CNN
-F 2 "kbd:CherryMX_Hotswap" H 13275 1400 50  0001 C CNN
+F 2 "kbd:MX-Alps-HS-1U" H 13275 1400 50  0001 C CNN
 F 3 "" H 13275 1400 50  0000 C CNN
 	1    13275 1400
@@
 F 0 "SW25" H 14125 1510 50  0000 C CNN
 F 1 "SW_PUSH" H 13975 1320 50  0000 C CNN
-F 2 "kbd:CherryMX_Hotswap" H 13975 1400 50  0001 C CNN
+F 2 "kbd:MX-Alps-HS-1U" H 13975 1400 50  0001 C CNN
 F 3 "" H 13975 1400 50  0000 C CNN
 	1    13975 1400
@@
 F 0 "SW26" H 14825 1510 50  0000 C CNN
 F 1 "SW_PUSH" H 14675 1320 50  0000 C CNN
-F 2 "kbd:CherryMX_Hotswap" H 14675 1400 50  0001 C CNN
+F 2 "kbd:MX-Alps-HS-1U" H 14675 1400 50  0001 C CNN
 F 3 "" H 14675 1400 50  0000 C CNN
 	1    14675 1400
@@
 F 0 "SW27" H 15525 1510 50  0000 C CNN
 F 1 "SW_PUSH" H 15375 1320 50  0000 C CNN
-F 2 "kbd:CherryMX_Hotswap" H 15375 1400 50  0001 C CNN
+F 2 "kbd:MX-Alps-HS-1U" H 15375 1400 50  0001 C CNN
 F 3 "" H 15375 1400 50  0000 C CNN
 	1    15375 1400
@@
 F 0 "SW22" H 12025 1510 50  0000 C CNN
 F 1 "SW_PUSH" H 11875 1320 50  0000 C CNN
-F 2 "kbd:CherryMX_Hotswap" H 11875 1400 50  0001 C CNN
+F 2 "kbd:MX-Alps-HS-1U" H 11875 1400 50  0001 C CNN
 F 3 "" H 11875 1400 50  0000 C CNN
 	1    11875 1400
@@
 F 0 "SW29" H 12725 2110 50  0000 C CNN
 F 1 "SW_PUSH" H 12575 1920 50  0000 C CNN
-F 2 "kbd:CherryMX_Hotswap" H 12575 2000 50  0001 C CNN
+F 2 "kbd:MX-Alps-HS-1U" H 12575 2000 50  0001 C CNN
 F 3 "" H 12575 2000 50  0000 C CNN
 	1    12575 2000
@@
 F 0 "SW30" H 13425 2110 50  0000 C CNN
 F 1 "SW_PUSH" H 13275 1920 50  0000 C CNN
-F 2 "kbd:CherryMX_Hotswap" H 13275 2000 50  0001 C CNN
+F 2 "kbd:MX-Alps-HS-1U" H 13275 2000 50  0001 C CNN
 F 3 "" H 13275 2000 50  0000 C CNN
 	1    13275 2000
@@
 F 0 "SW31" H 14125 2110 50  0000 C CNN
 F 1 "SW_PUSH" H 13975 1920 50  0000 C CNN
-F 2 "kbd:CherryMX_Hotswap" H 13975 2000 50  0001 C CNN
+F 2 "kbd:MX-Alps-HS-1U" H 13975 2000 50  0001 C CNN
 F 3 "" H 13975 2000 50  0000 C CNN
 	1    13975 2000
@@
 F 0 "SW32" H 14825 2110 50  0000 C CNN
 F 1 "SW_PUSH" H 14675 1920 50  0000 C CNN
-F 2 "kbd:CherryMX_Hotswap" H 14675 2000 50  0001 C CNN
+F 2 "kbd:MX-Alps-HS-1U" H 14675 2000 50  0001 C CNN
 F 3 "" H 14675 2000 50  0000 C CNN
 	1    14675 2000
@@
 F 0 "SW33" H 15525 2110 50  0000 C CNN
 F 1 "SW_PUSH" H 15375 1920 50  0000 C CNN
-F 2 "kbd:CherryMX_Hotswap" H 15375 2000 50  0001 C CNN
+F 2 "kbd:MX-Alps-HS-1U" H 15375 2000 50  0001 C CNN
 F 3 "" H 15375 2000 50  0000 C CNN
 	1    15375 2000
@@
 F 0 "SW28" H 12025 2110 50  0000 C CNN
 F 1 "SW_PUSH" H 11875 1920 50  0000 C CNN
-F 2 "kbd:CherryMX_Hotswap" H 11875 2000 50  0001 C CNN
+F 2 "kbd:MX-Alps-HS-1U" H 11875 2000 50  0001 C CNN
 F 3 "" H 11875 2000 50  0000 C CNN
 	1    11875 2000
@@
 F 0 "SW35" H 12725 2710 50  0000 C CNN
 F 1 "SW_PUSH" H 12575 2520 50  0000 C CNN
-F 2 "kbd:CherryMX_Hotswap" H 12575 2600 50  0001 C CNN
+F 2 "kbd:MX-Alps-HS-1U" H 12575 2600 50  0001 C CNN
 F 3 "" H 12575 2600 50  0000 C CNN
 	1    12575 2600
@@
 F 0 "SW36" H 13425 2710 50  0000 C CNN
 F 1 "SW_PUSH" H 13275 2520 50  0000 C CNN
-F 2 "kbd:CherryMX_Hotswap" H 13275 2600 50  0001 C CNN
+F 2 "kbd:MX-Alps-HS-1U" H 13275 2600 50  0001 C CNN
 F 3 "" H 13275 2600 50  0000 C CNN
 	1    13275 2600
@@
 F 0 "SW37" H 14125 2710 50  0000 C CNN
 F 1 "SW_PUSH" H 13975 2520 50  0000 C CNN
-F 2 "kbd:CherryMX_Hotswap" H 13975 2600 50  0001 C CNN
+F 2 "kbd:MX-Alps-HS-1U" H 13975 2600 50  0001 C CNN
 F 3 "" H 13975 2600 50  0000 C CNN
 	1    13975 2600
@@
 F 0 "SW38" H 14825 2710 50  0000 C CNN
 F 1 "SW_PUSH" H 14675 2520 50  0000 C CNN
-F 2 "kbd:CherryMX_Hotswap" H 14675 2600 50  0001 C CNN
+F 2 "kbd:MX-Alps-HS-1U" H 14675 2600 50  0001 C CNN
 F 3 "" H 14675 2600 50  0000 C CNN
 	1    14675 2600
@@
 F 0 "SW39" H 15525 2710 50  0000 C CNN
 F 1 "SW_PUSH" H 15375 2520 50  0000 C CNN
-F 2 "kbd:CherryMX_Hotswap" H 15375 2600 50  0001 C CNN
+F 2 "kbd:MX-Alps-HS-1U" H 15375 2600 50  0001 C CNN
 F 3 "" H 15375 2600 50  0000 C CNN
 	1    15375 2600
@@
 F 0 "SW34" H 12025 2710 50  0000 C CNN
 F 1 "SW_PUSH" H 11875 2520 50  0000 C CNN
-F 2 "kbd:CherryMX_Hotswap" H 11875 2600 50  0001 C CNN
+F 2 "kbd:MX-Alps-HS-1U" H 11875 2600 50  0001 C CNN
 F 3 "" H 11875 2600 50  0000 C CNN
 	1    11875 2600
@@
 F 0 "SW41" H 14825 3310 50  0000 C CNN
 F 1 "SW_PUSH" H 14675 3120 50  0000 C CNN
-F 2 "kbd:CherryMX_Hotswap" H 14675 3200 50  0001 C CNN
+F 2 "kbd:MX-Alps-HS-1U" H 14675 3200 50  0001 C CNN
 F 3 "" H 14675 3200 50  0000 C CNN
 	1    14675 3200
@@
 F 0 "SW42" H 15525 3310 50  0000 C CNN
 F 1 "SW_PUSH" H 15375 3120 50  0000 C CNN
-F 2 "kbd:CherryMX_Hotswap_1.5u" H 15375 3200 50  0001 C CNN
+F 2 "kbd:MX-Alps-HS-1.5U" H 15375 3200 50  0001 C CNN
 F 3 "" H 15375 3200 50  0000 C CNN
 	1    15375 3200
@@
 F 0 "SW40" H 14125 3310 50  0000 C CNN
 F 1 "SW_PUSH" H 13975 3120 50  0000 C CNN
-F 2 "kbd:CherryMX_Hotswap" H 13975 3200 50  0001 C CNN
+F 2 "kbd:MX-Alps-HS-1U" H 13975 3200 50  0001 C CNN
 F 3 "" H 13975 3200 50  0000 C CNN
 	1    13975 3200
@@
 F 0 "SW43" H 12025 3310 50  0000 C CNN
 F 1 "SW_PUSH" H 11875 3120 50  0000 C CNN
-F 2 "kbd:CherryMX_Hotswap" H 11875 3200 50  0001 C CNN
+F 2 "kbd:MX-Alps-HS-1U" H 11875 3200 50  0001 C CNN
 F 3 "" H 11875 3200 50  0000 C CNN
 	1    11875 3200
@@
 F 0 "J5" H 12503 3726 50  0000 L CNN
 F 1 "Conn_01x02_Female" H 12503 3635 50  0000 L CNN
-F 2 "Connector_PinHeader_2.00mm:PinHeader_1x02_P2.00mm_Vertical" H 12475 3750 50  0001 C CNN
+F 2 "kbd:Battery_Header" H 12475 3750 50  0001 C CNN
 F 3 "~" H 12475 3750 50  0001 C CNN
 	1    12475 3750
@@
 	12075 3850 12275 3850
 $Comp
-L power:GNDA #PWR?
+L power:GNDA #PWR0101
 U 1 1 60DE1EE2
 P 12275 3750
-F 0 "#PWR?" H 12275 3500 50  0001 C CNN
+F 0 "#PWR0101" H 12275 3500 50  0001 C CNN
 F 1 "GNDA" V 12280 3623 50  0000 R CNN
 F 2 "" H 12275 3750 50  0001 C CNN
